File: Board Files/549-addon.brd (EAGLE design)
At the start: 86.1 x 57.1 mm, 32 parts, among them P8_LEFT M23, P8_RIGHT M23, P9_LEFT M23, P9_RIGHT M23

Commit message: Updated schematic and layout to reflect changing pins for LEDs/buttons/buzzer
Parts:
- moved SG1 1.80 mm to (55.9, 36.8), turned to 180 degrees
- moved P8_LEFT 0.08 mm to (45.7, 50.2)
- turned R8 to 270 degrees
Connections:
- removed net N$10: P8_RIGHT.23, R4.2
- removed net N$5: P8_RIGHT.22, R5.2
- removed net N$6: P8_LEFT.24, R1.2
- removed net N$7: P8_LEFT.23, R3.2
- removed net N$8: P8_LEFT.22, R9.2
- removed net N$9: P8_RIGHT.24, R2.2
- new net LED1: P8_RIGHT.10, R1.2
- new net LED2: P8_LEFT.10, R2.2
- new net LED3: P8_RIGHT.9, R3.2
- new net LED4: P8_LEFT.9, R4.2
- new net LED5: P8_RIGHT.8, R5.2
- new net STATUSLED: P8_LEFT.8, R9.2
- net B0: now also P9_LEFT.8; no longer P8_RIGHT.3
- net B1: now also P9_RIGHT.8; no longer P8_LEFT.4
- net N$14: now also P9_RIGHT.7; no longer P8_RIGHT.21
- net RESETBUTTON: now also P8_RIGHT.14; no longer P8_LEFT.3
Routing:
- net STATUSLED: track 0.00 -> 56.5 mm
- net LED5: track 0.00 -> 52.8 mm
- net LED3: track 0.00 -> 47.1 mm
- net LED4: track 0.00 -> 46.9 mm
- net LED2: track 0.00 -> 40.5 mm
- net LED1: track 0.00 -> 40.0 mm
- net N$8: track 30.7 -> 0.00 mm
- net N$5: track 27.2 -> 0.00 mm
- net N$10: track 22.5 -> 0.00 mm, vias 1 -> 0
- net B1: track 21.8 -> 43.1 mm
- net N$14: track 21.6 -> 42.5 mm, vias 0 -> 1
- net N$9: track 16.0 -> 0.00 mm
- net B0: track 47.3 -> 31.3 mm, vias 1 -> 2
- net N$7: track 15.3 -> 0.00 mm, vias 1 -> 0
- net N$6: track 7.62 -> 0.00 mm
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Other:
- board text removed: "Arman is a suka"
- board text removed: "Bryan needs to calm down"
